File: vop24_lpcxpresso1769_basehw/Comunicacion.sch (KiCad schematic (older format))
At the start: 26 parts, among them J301 USB_B_Micro, J302 Screw_Terminal_01x02, U301 LTC4411, U302 TPD4S014, U303 LT1512

Commit message: actualizacion de PCB con cambios de ESQ
Parts:
- NT301, NT302: footprint NetTie:NetTie-2_THT_Pad1.0mm -> NetTie:NetTie-2_SMD_Pad0.5mm
- U302: footprint (none) -> Package_SON:Texas_S-PWSON-N10_ThermalVias
- U303: footprint (none) -> Package_SO:SO-8_5.3x6.2mm_P1.27mm
Changed lines of the file:
@@
 F 0 "U303" H 7100 3400 50  0000 C CNN
 F 1 "LT1512" H 6750 3400 50  0000 C CNN
-F 2 "" H 6600 3000 50  0001 C CNN
+F 2 "Package_SO:SO-8_5.3x6.2mm_P1.27mm" H 6600 3000 50  0001 C CNN
 F 3 "" H 6600 3000 50  0001 C CNN
 	1    6600 3000
@@
 F 0 "U302" H 3500 2965 50  0000 C CNN
 F 1 "TPD4S014" H 3500 2874 50  0000 C CNN
-F 2 "" H 3350 2500 50  0001 C CNN
+F 2 "Package_SON:Texas_S-PWSON-N10_ThermalVias" H 3350 2500 50  0001 C CNN
 F 3 "/home/froux/Dropbox/VOP24/docs y hojas de datos/otros/cosas modulo usb/tpd4s014.pdf" H 3350 2500 50  0001 C CNN
 	1    3500 2500
@@
 F 0 "NT302" H 5300 4428 50  0000 C CNN
 F 1 "Net-Tie_2" H 5300 4337 50  0000 C CNN
-F 2 "NetTie:NetTie-2_THT_Pad1.0mm" H 5300 4250 50  0001 C CNN
+F 2 "NetTie:NetTie-2_SMD_Pad0.5mm" H 5300 4250 50  0001 C CNN
 F 3 "~" H 5300 4250 50  0001 C CNN
 	1    5300 4250
@@
 F 0 "NT301" H 2250 6500 50  0000 C CNN
 F 1 "Net-Tie_2" H 2250 6400 50  0000 C CNN
-F 2 "NetTie:NetTie-2_THT_Pad1.0mm" H 2250 6450 50  0001 C CNN
+F 2 "NetTie:NetTie-2_SMD_Pad0.5mm" H 2250 6450 50  0001 C CNN
 F 3 "~" H 2250 6450 50  0001 C CNN
 	1    2250 6450

Commit message: ESQ: cambios en net-tie y footprints PCB: cambios grandes de dimensiones y ruteo
Parts:
- U302: footprint Package_SON:Texas_S-PWSON-N10_ThermalVias -> meport_kicad_libs:Texas_R-PWSON-N10
Changed lines of the file:
@@
 F 0 "U302" H 3500 2965 50  0000 C CNN
 F 1 "TPD4S014" H 3500 2874 50  0000 C CNN
-F 2 "Package_SON:Texas_S-PWSON-N10_ThermalVias" H 3350 2500 50  0001 C CNN
+F 2 "meport_kicad_libs:Texas_R-PWSON-N10" H 3350 2500 50  0001 C CNN
 F 3 "/home/froux/Dropbox/VOP24/docs y hojas de datos/otros/cosas modulo usb/tpd4s014.pdf" H 3350 2500 50  0001 C CNN
 	1    3500 2500
